File: PiCo2040-zero Новая плата управления экструдером/Плата управления экструдером PICI2040/Плата управления экструдером PICI2040.kicad_sch (KiCad schematic)
At the start: 29 parts, among them J10 Conn_01x08_Pin, J5 Conn_01x08_Pin, J6 Conn_01x08_Pin, J7 Conn_01x08_Pin, J8 Conn_01x08_Pin, J9 Conn_02x03_Odd_Even, Q1 IRLB8721, Q2 IRLB8721, Q3 IRLB8721, U1 rp2040-zero

Commit message: Разводка платы
Connections:
- net PB0 is gone; now on net j10_4: J10.4 (Pin_4)
- net PB1 is gone; now on net j10_5: J10.5 (Pin_5)
- net PB2 is gone; now on net j10_6: J10.6 (Pin_6)
- net PB3 is gone; now on net j10_7: J10.7 (Pin_7)
- net PB4 is gone; now on net j10_8: J10.8 (Pin_8)
- net PD5 is gone; now on net j10_1: J10.1 (Pin_1)
- net PD6 is gone; now on net j10_2: J10.2 (Pin_2)
- net PD7 is gone; now on net j10_3: J10.3 (Pin_3)
- net +3.3V: now also J7.2 (Pin_2)
- net BL_Z-min: now also U1.1 (0)
- net BL_contr_signal: now also U1.2 (1)
- net GND: now also J5.3 (Pin_3), J5.4 (Pin_4), J7.3 (Pin_3), J7.4 (Pin_4); no longer J6.6 (Pin_6), J8.6 (Pin_6)
- net cooler: now also U1.5 (4)
- net fan_control: now also U1.3 (2)
- net heater: now also U1.4 (3)
- net switch: now also U1.8 (7)
- net termistor: now also U1.7 (6)
- net rez_17: now reaches J5.8 (Pin_8)
- net rez_17: now also U1.17 (26)
- net j10_2: now reaches U1.10 (9)
- net j10_3: now reaches U1.11 (10)
- net j10_4: now reaches U1.12 (11)
- net j10_5: now reaches U1.13 (12)
- net j10_6: now reaches U1.14 (13)
- net j10_7: now reaches U1.15 (14)
- net j10_8: now reaches U1.16 (15)
- net rez_6: now reaches U1.6 (5)
- net rez_6: now also J6.6 (Pin_6)
- net j10_1: now reaches U1.9 (8)
- new net rez_6_PB: J8.6 (Pin_6)
- no-connect marks 0 -> 1
Other:
- moved on the sheet: J5

Commit message: Трассировка
Parts:
- added R10, R8, R9: 100R, Resistor_SMD:R_0805_2012Metric_Pad1.20x1.40mm_HandSolder, symbol Device:R
Connections:
- net +3.3V: now also R7.1
- net +5V: no longer R7.1
- net cooler_PB: now also R9.1; no longer Q2.1 (G), R4.1
- net fan_control: now also J6.6 (Pin_6), U1.6 (5); no longer J6.3 (Pin_3), U1.3 (2)
- net fan_control_PB: now also J8.6 (Pin_6), R10.1; no longer J8.3 (Pin_3), Q1.1 (G), R5.1
- net heater_PB: now also R8.1; no longer Q3.1 (G), R6.1
- net rez_17: now also J6.7 (Pin_7), U1.7 (6); no longer J5.8 (Pin_8), U1.17 (26)
- net rez_6: now also J6.3 (Pin_3), U1.3 (2); no longer J6.6 (Pin_6), U1.6 (5)
- net rez_6_PB: now also J8.3 (Pin_3); no longer J8.6 (Pin_6)
- net termistor: now also J5.8 (Pin_8), U1.17 (26); no longer J6.7 (Pin_7), U1.7 (6)
- net termistor_PB: now also J7.8 (Pin_8); no longer J8.7 (Pin_7)
- new net: Q3.1 (G), R6.1, R8.2
- new net: Q1.1 (G), R10.2, R5.1
- new net: Q2.1 (G), R4.1, R9.2
- new net rez_17_PB: J8.7 (Pin_7)
- no-connect marks 1 -> 0
Other:
- moved on the sheet: J10, J5, J6, J7, J8
