File: PiCo2040-zero Новая плата управления экструдером/Плата управления экструдером PICI2040/Плата управления экструдером PICI2040.kicad_pcb (KiCad board)
At the start: 2 copper layers, 100.2 x 42 mm, 29 parts, among them J10 Conn_01x08_Pin, J5 Conn_01x08_Pin, J6 Conn_01x08_Pin, J7 Conn_01x08_Pin, J8 Conn_01x08_Pin, J9 Conn_02x03_Odd_Even, Q1 IRLB8721, Q2 IRLB8721, Q3 IRLB8721, U1 rp2040-zero

Commit message: Разводка платы
Parts:
- moved R6 20.6 mm to (154.8, 67.8)
- moved Q2 3.80 mm to (136.8, 105.5)
- moved POWER_IN_24V1 1.12 mm to (109.7, 81.0)
- moved bl_touch1 0.98 mm to (130.5, 80.0)
- moved U1 0.63 mm to (181.0, 89.4)
- moved extruder1 0.62 mm to (116.5, 80.0)
Connections:
- J10 pad 1: /PD5 -> /j10_1
- J10 pad 2: /PD6 -> /j10_2
- J10 pad 3: /PD7 -> /j10_3
- J10 pad 4: /PB0 -> /j10_4
- J10 pad 5: /PB1 -> /j10_5
- J10 pad 6: /PB2 -> /j10_6
- J10 pad 7: /PB3 -> /j10_7
- J10 pad 8: /PB4 -> /j10_8
- J5 pad 3: unconnected-(J5-Pin_3-Pad3) -> GND
- J5 pad 4: unconnected-(J5-Pin_4-Pad4) -> GND
- J5 pad 8: unconnected-(J5-Pin_8-Pad8) -> /rez_17
- J6 pad 6: GND -> /rez_6
- J7 pad 2: unconnected-(J7-Pin_2-Pad2) -> +3.3V
- J7 pad 3: unconnected-(J7-Pin_3-Pad3) -> GND
- J7 pad 4: unconnected-(J7-Pin_4-Pad4) -> GND
- J8 pad 6: GND -> /rez_6_PB
- U1 pad 1: unconnected-(U1-0-Pad1) -> /BL_Z-min
- U1 pad 10: unconnected-(U1-9-Pad10) -> /j10_2
- U1 pad 11: unconnected-(U1-10-Pad11) -> /j10_3
- U1 pad 12: unconnected-(U1-11-Pad12) -> /j10_4
- U1 pad 13: unconnected-(U1-12-Pad13) -> /j10_5
- U1 pad 14: unconnected-(U1-13-Pad14) -> /j10_6
- U1 pad 15: unconnected-(U1-14-Pad15) -> /j10_7
- U1 pad 16: unconnected-(U1-15-Pad16) -> /j10_8
- U1 pad 17: unconnected-(U1-26-Pad17) -> /rez_17
- U1 pad 2: unconnected-(U1-1-Pad2) -> /BL_contr_signal
- U1 pad 3: unconnected-(U1-2-Pad3) -> /fan_control
- U1 pad 4: unconnected-(U1-3-Pad4) -> /heater
- U1 pad 5: unconnected-(U1-4-Pad5) -> /cooler
- U1 pad 6: unconnected-(U1-5-Pad6) -> /rez_6
- U1 pad 7: unconnected-(U1-6-Pad7) -> /termistor
- U1 pad 8: unconnected-(U1-7-Pad8) -> /switch
- U1 pad 9: unconnected-(U1-8-Pad9) -> /j10_1
Routing:
- net +3.3V: track 0.00 -> 42.0 mm
- net /j10_8: track 0.00 -> 24.9 mm
- net Net-(Q2-D): track 0.00 -> 21.1 mm
- net /j10_3: track 0.00 -> 19.2 mm
- net /rez_17: track 0.00 -> 19.1 mm
- net /j10_5: track 0.00 -> 18.8 mm
- net /j10_6: track 0.00 -> 18.5 mm
- net /j10_4: track 0.00 -> 18.5 mm
- net /j10_7: track 0.00 -> 18.5 mm
- net /j10_2: track 0.00 -> 18.5 mm
- net /j10_1: track 0.00 -> 18.5 mm
- net /DIR: track 0.00 -> 18.4 mm
- net /STEP: track 0.00 -> 18.4 mm
- net /ENABLE: track 0.77 -> 19.1 mm
- net +5V: track 39.4 -> 56.7 mm
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
Commit message: Трассировка
Parts:
- added R10: 100R, Resistor_SMD:R_0805_2012Metric_Pad1.20x1.40mm_HandSolder, F.Cu at (137.5, 102.4)
- added R8: 100R, Resistor_SMD:R_0805_2012Metric_Pad1.20x1.40mm_HandSolder, F.Cu at (137.5, 97.3)
- added R9: 100R, Resistor_SMD:R_0805_2012Metric_Pad1.20x1.40mm_HandSolder, F.Cu at (137.5, 99.8)
- R7: moved to B.Cu
- moved R6 35.4 mm to (133.5, 96.1), turned to 90 degrees
- moved R7 31.0 mm to (104.3, 111.0)
- moved R4 26.0 mm to (133.5, 101.3), turned to -90 degrees
- moved fan1 25.4 mm to (132.6, 116.7)
- moved term1 25.4 mm to (107.1, 116.7)
- moved Q3 25.4 mm to (113.7, 107.6)
- moved R5 25.0 mm to (137.5, 104.7), turned to 0 degrees
- moved C11 21.0 mm to (108.4, 104.7), turned to 0 degrees
- moved Q1 16.0 mm to (136.5, 107.6)
- moved Q2 11.9 mm to (125.1, 107.6)
- moved A1 2.40 mm to (127.5, 87.4)
Connections:
- J5 pad 8: /rez_17 -> /termistor
- J6 pad 3: /fan_control -> /rez_6
- J6 pad 6: /rez_6 -> /fan_control
- J6 pad 7: /termistor -> /rez_17
- J7 pad 8: unconnected-(J7-Pin_8-Pad8) -> /termistor_PB
- J8 pad 3: /fan_control_PB -> /rez_6_PB
- J8 pad 6: /rez_6_PB -> /fan_control_PB
- J8 pad 7: /termistor_PB -> /rez_17_PB
- Q1 pad 1: /fan_control_PB -> Net-(Q1-G)
- Q2 pad 1: /cooler_PB -> Net-(Q2-G)
- Q3 pad 1: /heater_PB -> Net-(Q3-G)
- R4 pad 1: /cooler_PB -> Net-(Q2-G)
- R5 pad 1: /fan_control_PB -> Net-(Q1-G)
- R6 pad 1: /heater_PB -> Net-(Q3-G)
- R7 pad 1: +5V -> +3.3V
- U1 pad 17: /rez_17 -> /termistor
- U1 pad 3: /fan_control -> /rez_6
- U1 pad 6: /rez_6 -> /fan_control
- U1 pad 7: /termistor -> /rez_17
Routing:
- net +24V: track 0.00 -> 34.6 mm
- net Net-(Q3-G): track 0.00 -> 27.1 mm
- net +3.3V: track 42.0 -> 64.0 mm
- net Net-(Q2-G): track 0.00 -> 14.6 mm
- net Net-(Q2-D): track 21.1 -> 9.51 mm
- net Net-(Q1-D): track 0.00 -> 10.7 mm
- net Net-(Q3-D): track 0.00 -> 9.94 mm
- net Net-(Q1-G): track 0.00 -> 5.21 mm
- net /termistor: track 15.7 -> 19.1 mm
- net /rez_17: track 19.1 -> 15.7 mm
- net /fan_control_PB: track 0.00 -> 3.32 mm
- net /cooler_PB: track 0.00 -> 3.31 mm
- net /heater_PB: track 0.00 -> 3.31 mm
- net /BL_contr_signal_PB: track 14.0 -> 17.1 mm
- net /ENABLE_PB: track 3.62 -> 6.19 mm
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- added copper zone on B.Cu, net GND
- added copper zone on F.Cu, net GND

Commit message: Мелкие правки платы
Parts:
- moved J9 5.73 mm to (124.4, 91.1)
- moved A1 1.51 mm to (126.0, 87.4)
Routing:
- net GND: track 0.04 -> 20.5 mm
- net Net-(A1-MS3): track 5.05 -> 11.3 mm
- net Net-(A1-MS1): track 12.2 -> 18.3 mm
- net Net-(A1-MS2): track 8.64 -> 14.7 mm
- net +3.3V: track 64.0 -> 61.9 mm
- net /DIR_PB: track 25.7 -> 24.2 mm
- net /STEP_PB: track 22.1 -> 20.6 mm
- net /ENABLE_PB: track 6.19 -> 4.69 mm
- net /BL_contr_signal_PB: track 17.1 -> 15.9 mm
- net Net-(A1-2A): track 7.64 -> 8.26 mm
- net Net-(A1-1B): track 7.60 -> 8.23 mm
- net Net-(A1-2B): track 7.65 -> 8.28 mm
- net Net-(A1-1A): track 7.62 -> 8.25 mm

Commit message: Механика гравера
Routing:
- net +3.3V: track 61.9 -> 66.9 mm
Changed lines of the file:
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@@
+	)
+	(segment
+		(start 126.965 91.06)
+		(end 126.965 93.6)
+		(width 0.5)
+		(layer "F.Cu")
+		(net "+3.3V")
 	)
 	(segment
@@
 		(width 0.5)
 		(layer "F.Cu")
+		(net "+3.3V")
+	)
+	(segment
+		(start 126.965 93.6)
+		(end 126.965 96.14)
+		(width 0.5)
+		(layer "F.Cu")
